Commit message: Release Version 1.0.0

File: safemotions/description/urdf/one_robot.urdf (robot description, URDF)
Before this commit: robot main, 12 links, 11 joints
Links:
- removed link iiwa_link_ee
Joints:
- removed joint iiwa_joint_ee

File: safemotions/description/urdf/three_robots.urdf (robot description, URDF)
Before this commit: robot main, 32 links, 31 joints
Links:
- removed link iiwa_link_ee_r0
- removed link iiwa_link_ee_r1
- removed link iiwa_link_ee_r2
Joints:
- removed joint iiwa_joint_ee_r0
- removed joint iiwa_joint_ee_r1
- removed joint iiwa_joint_ee_r2

File: safemotions/description/urdf/two_robots.urdf (robot description, URDF)
Before this commit: robot main, 22 links, 21 joints
Links:
- removed link iiwa_link_ee_r0
- removed link iiwa_link_ee_r1
Joints:
- removed joint iiwa_joint_ee_r0
- removed joint iiwa_joint_ee_r1
